Commit message: integration with orunav

File: velodyne_description/urdf/VLP-16.urdf.xacro (robot description, xacro)
@@ -2,5 +2,5 @@
 <robot xmlns:xacro="http://www.ros.org/wiki/xacro" name="VLP-16">
   <xacro:property name="M_PI" value="3.1415926535897931" />
-  <xacro:macro name="VLP-16" params="*origin parent:=base_link name:=velodyne topic:=/velodyne_points hz:=10 lasers:=16 samples:=1875 collision_range:=0.3 min_range:=0.9 max_range:=130.0 noise:=0.008 min_angle:=-${M_PI} max_angle:=${M_PI}">
+  <xacro:macro name="VLP-16" params="*origin parent:=base_link prefix=no_prefix name:=velodyne topic:=/velodyne_points hz:=10 lasers:=16 samples:=1875 collision_range:=0.3 min_range:=0.9 max_range:=30.0 noise:=0.008 min_angle:=-${M_PI} max_angle:=${M_PI}">
     <joint name="${name}_base_mount_joint" type="fixed">
       <xacro:insert_block name="origin" />
@@ -83,5 +83,5 @@
         <plugin name="gazebo_ros_laser_controller" filename="libgazebo_ros_velodyne_laser.so">
           <topicName>${topic}</topicName>
-          <frameName>/${name}</frameName>
+          <frameName>/${prefix}/${name}</frameName>
           <min_range>${min_range}</min_range>
           <max_range>${max_range}</max_range>

File: velodyne_description/urdf/example2.urdf.xacro (robot description, xacro)
@@ -4,8 +4,14 @@
   <link name="base_footprint" />
   <!-- Base Link -->
+  <link name="world"/>
+  <joint name="worldjoint" type="fixed" >
+   <parent link="world" />
+    <child link="base_footprint" />
+    <origin xyz="0 0 1.7" rpy="0 0 0" />
+  </joint>
   <joint name="footprint" type="fixed" >
    <parent link="base_footprint" />
     <child link="base_link" />
-    <origin xyz="0 0 0.05" rpy="0 0 0" />
+    <origin xyz="0 0 0.4" rpy="0 0 0" />
   </joint>
   <link name="base_link" >
@@ -30,5 +36,5 @@
   <xacro:include filename="$(find velodyne_description)/urdf/VLP-16.urdf.xacro"/>
   <VLP-16 parent="base_link" name="velodyne" topic="/velodyne_points" hz="10" samples="440">
-    <origin xyz="0 0 4" rpy="0 0 0" />
+    <origin xyz="0 0 0.4" rpy="0 0 0" />
   </VLP-16>
   <!--xacro:include filename="$(find velodyne_description)/urdf/HDL-32E.urdf.xacro"/>

Commit message: fixed topic prefix for velodyne

File: velodyne_description/urdf/VLP-16.urdf.xacro (robot description, xacro)
@@ -2,5 +2,5 @@
 <robot xmlns:xacro="http://www.ros.org/wiki/xacro" name="VLP-16">
   <xacro:property name="M_PI" value="3.1415926535897931" />
-  <xacro:macro name="VLP-16" params="*origin parent:=base_link prefix=no_prefix name:=velodyne topic:=/velodyne_points hz:=10 lasers:=16 samples:=1875 collision_range:=0.3 min_range:=0.9 max_range:=30.0 noise:=0.008 min_angle:=-${M_PI} max_angle:=${M_PI}">
+  <xacro:macro name="VLP-16" params="*origin parent:=base_link prefix=robot1 name:=velodyne topic:=/velodyne_points hz:=10 lasers:=16 samples:=1875 collision_range:=0.3 min_range:=0.9 max_range:=30.0 noise:=0.008 min_angle:=-${M_PI} max_angle:=${M_PI}">
     <joint name="${name}_base_mount_joint" type="fixed">
       <xacro:insert_block name="origin" />
@@ -82,5 +82,5 @@
         </ray>
         <plugin name="gazebo_ros_laser_controller" filename="libgazebo_ros_velodyne_laser.so">
-          <topicName>${topic}</topicName>
+          <topicName>/${prefix}/${topic}</topicName>
           <frameName>/${prefix}/${name}</frameName>
           <min_range>${min_range}</min_range>
